File: PCB/RF_R1_8-9Xu.kicad_sch (KiCad schematic)
At the start: 37 parts, among them J1 JST, J2 JST, J3 Conn_01x03, J4 Conn_01x03, SW1 BOOT0, U1 STM32F401CBUx, U2 SN74AHCT1G125, U3 ME6206A33M3G, Y1 8 MHz

Commit message: Updated sheets
Other:
- company: Cipulot PCB Design  -> LU.SV Solutions

Commit message: Rev 1.2
Parts:
- C1: renamed from C15; MPN (none) -> CC0603KRX7R9BB104
- C10: renamed from C9; MPN (none) -> CL05B104KB54PNC
- C11: renamed from C10; MPN (none) -> CL05A105KA5NQNC
- C2: renamed from C1; MPN (none) -> CC0603KRX7R9BB104
- C3: renamed from C2; MPN (none) -> CL05A475MP5NRNC
- C4: renamed from C3; MPN (none) -> CL05A105KA5NQNC
- C5: renamed from C4; MPN (none) -> CL05A105KA5NQNC
- C6: renamed from C5; MPN (none) -> CL05B104KB54PNC
- C7: renamed from C6; MPN (none) -> CL05B104KB54PNC
- C8: renamed from C7; MPN (none) -> CL05B104KB54PNC
- C9: renamed from C8; MPN (none) -> CL05B104KB54PNC
- D1: MPN (none) -> PRTR5V0U2X
- F1: MPN (none) -> nSMD050-24V
- J1: MPN (none) -> S4B-EH(LF)(SN)
- J2: LCSC C145956 -> C160404; MPN (none) -> SM04B-SRSS-TB(LF)(SN)
- L1: MPN (none) -> BLM18KG331SN1D
- R1: renamed from R33; MPN (none) -> 0603WAF3300T5E
- R10: renamed from R9; MPN (none) -> 0402WGF1000TCE
- R11: renamed from R10; MPN (none) -> 0402WGF1002TCE
- R12: renamed from R11; MPN (none) -> 0402WGF1002TCE
- R13: renamed from R12; MPN (none) -> 0402WGF1002TCE
- R2: renamed from R1; MPN (none) -> 0402WGF5101TCE
- R3: renamed from R2; MPN (none) -> 0402WGF5101TCE
- R4: renamed from R3; MPN (none) -> 0402WGF1000TCE
- R5: renamed from R4; MPN (none) -> 0402WGF1000TCE
- R6: renamed from R5; MPN (none) -> 0402WGF1003TCE
- R7: renamed from R6; MPN (none) -> 0402WGF1000TCE
- R8: renamed from R7; MPN (none) -> 0402WGF1000TCE
- R9: renamed from R8; MPN (none) -> 0402WGF1000TCE
- U1: MPN (none) -> C118825
- U2: MPN (none) -> SN74AHCT1G125DBVR
- U3: MPN (none) -> ME6206A33M3G
- USB1: MPN (none) -> TYPE-C-31-M-12
- Y1: LCSC C907975 -> C341525; MPN (none) -> CSTNE8M00GH5C000R0
