File: PCB/analog.kicad_sch (KiCad schematic)
At the start: 26 parts, among them U4 74HC4051, U5 OPA350, U6 74HC4051

Commit message: Updated sheets
Other:
- company: Cipulot PCB Design  -> LU.SV Solutions
- title: RF_R1_8-9Xu PCB - Analog Circuit -> RF_R1_8-9Xu PCB

Commit message: Rev 1.2
Parts:
- removed C12: 220p, Capacitor_SMD:C_0603_1608Metric, symbol Device:C
- removed C13: 100n, Capacitor_SMD:C_0402_1005Metric, symbol Device:C
- removed R21: 100k, Resistor_SMD:R_0603_1608Metric, symbol Device:R
- removed R22: 1k, Resistor_SMD:R_0603_1608Metric, symbol Device:R
- removed U5: OPA350, Package_SO:SOIC-8_3.9x4.9mm_P1.27mm, symbol burrbrown:OPA350
- added C14: 220p, Capacitor_SMD:C_0603_1608Metric, symbol Device:C
- added C7: 100n, Resistor_SMD:R_0603_1608Metric, symbol Device:C
- added R10: 100k, Resistor_SMD:R_0603_1608Metric, symbol Device:R
- added R23: 1k, Resistor_SMD:R_0603_1608Metric, symbol Device:R
- added U3: OPA340NA, Package_TO_SOT_SMD:SOT-23-5, symbol Amplifier_Operational:OPA340NA
- C12: renamed from C11; MPN (none) -> CL05B104KB54PNC
- C15: renamed from C14; MPN (none) -> CL05B104KB54PNC
- JP1: footprint Resistor_SMD:R_0603_1608Metric -> Resistor_SMD:R_0603_1608Metric_Pad0.98x0.95mm_HandSolder
- R14: renamed from R13; MPN (none) -> 0402WGF1003TCE
- R15: renamed from R14; MPN (none) -> 0402WGF1003TCE
- R16: renamed from R15; MPN (none) -> 0402WGF1003TCE
- R17: renamed from R16; MPN (none) -> 0402WGF1003TCE
- R18: renamed from R17; MPN (none) -> 0402WGF1003TCE
- R19: renamed from R18; MPN (none) -> 0402WGF1003TCE
- R20: renamed from R19; MPN (none) -> 0402WGF1003TCE
- R21: renamed from R20; MPN (none) -> 0402WGF1003TCE
- R24: renamed from R23; MPN (none) -> 0402WGF1003TCE
- R25: renamed from R24; MPN (none) -> 0402WGF1003TCE
- R26: renamed from R25; MPN (none) -> 0402WGF1003TCE
- R27: renamed from R26; MPN (none) -> 0402WGF1003TCE
- R28: renamed from R27; MPN (none) -> 0402WGF1003TCE
- R29: renamed from R28; MPN (none) -> 0402WGF1003TCE
- R30: renamed from R29; MPN (none) -> 0402WGF1003TCE
- R31: renamed from R30; MPN (none) -> 0402WGF1003TCE
- U4, U6: value 74HC4051 -> CD74HC4051PWR; LCSC C5645 -> C352826; MPN (none) -> CD74HC4051PWR
Connections:
- net +3V3: now also C7.2, U3.5 (V+)
- net ADC: now also R10.2, U3.1
- net APLEX_OUT_PIN_0: now also C14.1, U3.3 (+)
- net GND: now also C14.2, C7.1, R23.2, U3.2 (V-)
- net at JP1.2 (B): now also R10.1, R23.1, U3.4 (-)
Other:
- note added: "Possible CN alternative: LCSC: C565341 MPN: OPA340M5/TR"
