File: PCB/indicators.kicad_sch (KiCad schematic)
At the start: 5 parts

Commit message: Updated sheets
Other:
- company: Cipulot PCB Design  -> LU.SV Solutions
- title: (none) -> RF_R1_8-9Xu PCB

Commit message: Rev 1.2
Parts:
- R32: renamed from R31; MPN (none) -> 0402WGF1000TCE
- R33: renamed from R32; MPN (none) -> 0402WGF1000TCE
Changed lines of the file:
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@@
   (title_block
     (title "RF_R1_8-9Xu PCB")
-    (date "2023-11-17")
-    (rev "1.1")
+    (date "2023-11-23")
+    (rev "1.2")
     (company "LU.SV Solutions")
     (comment 1 "Cipulot PCB Design")
@@
   (symbol (lib_id "Device:R") (at 100.965 57.15 180) (unit 1)
     (in_bom yes) (on_board yes) (dnp no)
-    (property "Reference" "R32" (at 103.505 57.15 0)
+    (property "Reference" "R33" (at 103.505 57.15 0)
       (effects (font (size 1.27 1.27)))
     )
@@
       (effects (font (size 1.27 1.27)) hide)
     )
-    (pin "1")
-    (pin "2")
-    (instances
-      (project "RF_R1_8-9Xu"
-        (path "/e63e39d7-6ac0-4ffd-8aa3-1841a4541b55/eb02aace-817b-4a3c-af71-6f158a79d714"
-          (reference "R32") (unit 1)
+    (property "MPN" "0402WGF1000TCE" (at 100.965 57.15 0)
+      (effects (font (size 1.27 1.27)) hide)
+    )
+    (pin "1")
+    (pin "2")
+    (instances
+      (project "RF_R1_8-9Xu"
+        (path "/e63e39d7-6ac0-4ffd-8aa3-1841a4541b55/eb02aace-817b-4a3c-af71-6f158a79d714"
+          (reference "R33") (unit 1)
         )
       )
@@
   (symbol (lib_id "power:GND") (at 100.965 73.66 0) (unit 1)
     (in_bom yes) (on_board yes) (dnp no) (fields_autoplaced)
-    (property "Reference" "#PWR069" (at 100.965 80.01 0)
+    (property "Reference" "#PWR072" (at 100.965 80.01 0)
       (effects (font (size 1.27 1.27)) hide)
     )
@@
       (project "RF_R1_8-9Xu"
         (path "/e63e39d7-6ac0-4ffd-8aa3-1841a4541b55/eb02aace-817b-4a3c-af71-6f158a79d714"
-          (reference "#PWR069") (unit 1)
+          (reference "#PWR072") (unit 1)
         )
       )
@@
   (symbol (lib_id "power:GND") (at 72.39 73.66 0) (unit 1)
     (in_bom yes) (on_board yes) (dnp no) (fields_autoplaced)
-    (property "Reference" "#PWR068" (at 72.39 80.01 0)
+    (property "Reference" "#PWR071" (at 72.39 80.01 0)
       (effects (font (size 1.27 1.27)) hide)
     )
@@
       (project "RF_R1_8-9Xu"
         (path "/e63e39d7-6ac0-4ffd-8aa3-1841a4541b55/eb02aace-817b-4a3c-af71-6f158a79d714"
-          (reference "#PWR068") (unit 1)
+          (reference "#PWR071") (unit 1)
         )
       )
@@
   (symbol (lib_id "Device:R") (at 72.39 57.15 180) (unit 1)
     (in_bom yes) (on_board yes) (dnp no)
-    (property "Reference" "R31" (at 74.93 57.15 0)
+    (property "Reference" "R32" (at 74.93 57.15 0)
       (effects (font (size 1.27 1.27)))
     )
@@
       (effects (font (size 1.27 1.27)) hide)
     )
-    (pin "1")
-    (pin "2")
-    (instances
-      (project "RF_R1_8-9Xu"
-        (path "/e63e39d7-6ac0-4ffd-8aa3-1841a4541b55/eb02aace-817b-4a3c-af71-6f158a79d714"
-          (reference "R31") (unit 1)
-        )
-      )
+    (property "MPN" "0402WGF1000TCE" (at 72.39 57.15 0)
+      (effects (font (size 1.27 1.27)) hide)
+    )
+    (pin "1")
+    (pin "2")
+    (instances
+      (project "RF_R1_8-9Xu"
+        (path "/e63e39d7-6ac0-4ffd-8aa3-1841a4541b55/eb02aace-817b-4a3c-af71-6f158a79d714"
+          (reference "R32") (unit 1)
+        )
+      )
