File: PCB/matrix.kicad_sch (KiCad schematic)
At the start: 99 parts, among them SW10 EC_SW, SW100 EC_SW, SW11 EC_SW, SW12 EC_SW, SW13 EC_SW, SW14 EC_SW, SW15 EC_SW, SW16 EC_SW, SW17 EC_SW, SW18 EC_SW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

Commit message: Updated sheets
Other:
- company: Cipulot PCB Design  -> LU.SV Solutions
- title: RF_R1_8-9Xu PCB - Matrix -> RF_R1_8-9Xu PCB
