File: PCB/mounting.kicad_sch (KiCad schematic)
At the start: 45 parts

Commit message: Updated sheets
Other:
- company: Cipulot PCB Design  -> LU.SV Solutions
- title: RF_R1_8-9Xu PCB - Mounting Points -> RF_R1_8-9Xu PCB
